File: kicad/Tlalocohyla_Smithii.kicad_pcb (KiCad board)
At the start: 2 copper layers, 215.7 x 90 mm, 74 parts

Commit message: Change Xiao footprint
Reset and Battery plus
Parts:
- removed the H** at (150.0, 80.0)
- removed PAD1, PAD2, PAD3, PAD4: , SMDPad
- Ref**: footprint Library:XiaoSimple -> Library:Xiao BLE pogo pins
- moved Ref** 13.5 mm to (150.0, 86.8), turned to 90 degrees
Connections:
- JST1 pad 1: JSTplus -> GND_XIAO
- JST1 pad 2: Bminus -> JSTplus
- Ref** pad 13: (no net) -> GND_XIAO
Routing:
- net Bminus: track 47.6 -> 0.00 mm
- net GND_XIAO: track 46.5 -> 85.9 mm
- net RST_XIAO: track 47.9 -> 59.0 mm, vias 1 -> 3
- net Bplus: track 66.6 -> 58.6 mm, vias 1 -> 3
- net JSTplus: track 37.9 -> 40.9 mm
- net P3: track 247.5 -> 248.4 mm

Commit message: Adjust tracks
Routing:
- net GND_XIAO: track 85.9 -> 85.0 mm
Changed lines of the file:
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@@
     (fp_arc (start 2.794 6.9088) (mid 2.7432 6.858) (end 2.794 6.8072) (layer "Dwgs.User") (width 0.1))
     (fp_arc (start -7.088 -6.8228) (mid -7.15135 -6.85665) (end -7.1175 -6.92) (layer "Dwgs.User") (width 0.1))
-    (fp_arc (start 3.0523 -6.922) (mid 3.107895 -6.87646) (end 3.0623 -6.8209) (layer "Dwgs.User") (width 0.1))
+    (fp_arc (start 3.0523 -6.922) (mid 3.107905 -6.87645) (end 3.0623 -6.8209) (layer "Dwgs.User") (width 0.1))
     (fp_arc (start -0.4797 -7.4055) (mid -0.44585 -7.46885) (end -0.3825 -7.435) (layer "Dwgs.User") (width 0.1))
     (fp_arc (start -2.4173 6.922) (mid -2.47285 6.87645) (end -2.4273 6.8209) (layer "Dwgs.User") (width 0.1))
@@
     (fp_arc (start -4.1658 -7.0304) (mid -4.2373 -7.0233) (end -4.2444 -7.0948) (layer "Dwgs.User") (width 0.1))
     (fp_arc (start 5.9942 -7.0304) (mid 5.9227 -7.0233) (end 5.9156 -7.0948) (layer "Dwgs.User") (width 0.1))
-    (fp_arc (start 7.2395 -7.4252) (mid 7.193905 -7.3696) (end 7.1384 -7.4152) (layer "Dwgs.User") (width 0.1))
-    (fp_arc (start 3.5555 7.4252) (mid 3.60105 7.369705) (end 3.6566 7.4152) (layer "Dwgs.User") (width 0.1))
+    (fp_arc (start 7.2395 -7.4252) (mid 7.193995 -7.3697) (end 7.1384 -7.4152) (layer "Dwgs.User") (width 0.1))
+    (fp_arc (start 3.5555 7.4252) (mid 3.601059 7.369695) (end 3.6566 7.4152) (layer "Dwgs.User") (width 0.1))
     (fp_arc (start -3.0353 7.5565) (mid -2.9845 7.5057) (end -2.9337 7.5565) (layer "Dwgs.User") (width 0.1))
     (fp_arc (start -9.5352 5.6354) (mid -9.57115 5.63535) (end -9.5711 5.5994) (layer "Dwgs.User") (width 0.1))
@@
     (fp_arc (start -7.0977 6.8209) (mid -7.05215 6.87645) (end -7.1077 6.922) (layer "Dwgs.User") (width 0.1))
     (fp_arc (start -1.9156 6.956) (mid -1.93645 6.88725) (end -1.8677 6.8664) (layer "Dwgs.User") (width 0.1))
-    (fp_arc (start 8.6355 7.4252) (mid 8.681005 7.3697) (end 8.7366 7.4152) (layer "Dwgs.User") (width 0.1))
+    (fp_arc (start 8.6355 7.4252) (mid 8.681095 7.3696) (end 8.7366 7.4152) (layer "Dwgs.User") (width 0.1))
     (fp_arc (start 7.1247 -8.89) (mid 7.1755 -8.9408) (end 7.2263 -8.89) (layer "Dwgs.User") (width 0.1))
     (fp_arc (start 4.8079 -7.0233) (mid 4.8008 -7.0948) (end 4.8723 -7.1019) (layer "Dwgs.User") (width 0.1))
@@
     (fp_arc (start -2.281 -6.9086) (mid -2.2354 -6.853) (end -2.291 -6.8074) (layer "Dwgs.User") (width 0.1))
     (fp_arc (start -8.8515 3.7081) (mid -8.8769 3.6827) (end -8.8515 3.6573) (layer "Dwgs.User") (width 0.1))
-    (fp_arc (start 5.2027 6.922) (mid 5.1471 6.876405) (end 5.1927 6.8209) (layer "Dwgs.User") (width 0.1))
+    (fp_arc (start 5.2027 6.922) (mid 5.1472 6.876495) (end 5.1927 6.8209) (layer "Dwgs.User") (width 0.1))
     (fp_arc (start 3.4471 7.0233) (mid 3.4542 7.0948) (end 3.3827 7.1019) (layer "Dwgs.User") (width 0.1))
     (fp_arc (start -4.064 5.9703) (mid -3.885316 6.044316) (end -3.8113 6.223) (layer "Dwgs.User") (width 0.1))
@@
     (fp_arc (start -8.6312 5.5369) (mid -8.6058 5.5623) (end -8.6312 5.5877) (layer "Dwgs.User") (width 0.1))
     (fp_arc (start 5.7523 -6.8664) (mid 5.683621 -6.887261) (end 5.7044 -6.956) (layer "Dwgs.User") (width 0.1))
-    (fp_arc (start 8.1323 -6.922) (mid 8.1879 -6.876405) (end 8.1423 -6.8209) (layer "Dwgs.User") (width 0.1))
+    (fp_arc (start 8.1323 -6.922) (mid 8.1878 -6.876495) (end 8.1423 -6.8209) (layer "Dwgs.User") (width 0.1))
     (fp_arc (start -8.6058 5.8928) (mid -8.6312 5.9182) (end -8.6566 5.8928) (layer "Dwgs.User") (width 0.1))
     (fp_arc (start 5.461 -6.9088) (mid 5.5118 -6.858) (end 5.461 -6.8072) (layer "Dwgs.User") (width 0.1))
@@
     (fp_arc (start -4.064 -6.4757) (mid -3.885316 -6.401684) (end -3.8113 -6.223) (layer "Dwgs.User") (width 0.1))
     (fp_arc (start -3.8087 6.223) (mid -3.883477 6.403523) (end -4.064 6.4783) (layer "Dwgs.User") (width 0.1))
-    (fp_arc (start 4.6995 -7.4252) (mid 4.653905 -7.3696) (end 4.5984 -7.4152) (layer "Dwgs.User") (width 0.1))
+    (fp_arc (start 4.6995 -7.4252) (mid 4.653995 -7.3697) (end 4.5984 -7.4152) (layer "Dwgs.User") (width 0.1))
     (fp_arc (start -3.0353 -8.89) (mid -2.9845 -8.9408) (end -2.9337 -8.89) (layer "Dwgs.User") (width 0.1))
     (fp_arc (start -9.652 4.318) (mid -9.831603 4.243603) (end -9.906 4.064) (layer "Dwgs.User") (width 0.1))
-    (fp_arc (start 6.0955 7.4252) (mid 6.141095 7.3696) (end 6.1966 7.4152) (layer "Dwgs.User") (width 0.1))
+    (fp_arc (start 6.0955 7.4252) (mid 6.141005 7.3697) (end 6.1966 7.4152) (layer "Dwgs.User") (width 0.1))
     (fp_arc (start 2.1935 7.3131) (mid 2.124761 7.333979) (end 2.1039 7.2652) (layer "Dwgs.User") (width 0.1))
     (fp_arc (start -2.0277 -6.922) (mid -1.97215 -6.87645) (end -2.0177 -6.8209) (layer "Dwgs.User") (width 0.1))
@@
     (fp_arc (start -1.4253 7.4055) (mid -1.45915 7.46885) (end -1.5225 7.435) (layer "Dwgs.User") (width 0.1))
     (fp_arc (start -3.9499 7.5515) (mid -3.9955 7.6071) (end -4.0511 7.5615) (layer "Dwgs.User") (width 0.1))
-    (fp_arc (start 7.7427 6.922) (mid 7.6872 6.876495) (end 7.7327 6.8209) (layer "Dwgs.User") (width 0.1))
+    (fp_arc (start 7.7427 6.922) (mid 7.6871 6.876405) (end 7.7327 6.8209) (layer "Dwgs.User") (width 0.1))
     (fp_arc (start 2.5414 6.9598) (mid 2.4781 6.9259) (end 2.512 6.8626) (layer "Dwgs.User") (width 0.1))
     (fp_arc (start -9.2203 5.8557) (mid -9.2203 5.8198) (end -9.1844 5.8198) (layer "Dwgs.User") (width 0.1))
@@
     (fp_arc (start 0.9777 7.3039) (mid 1.0116 7.2406) (end 1.0749 7.2745) (layer "Dwgs.User") (width 0.1))
     (fp_arc (start -0.0373 6.8664) (mid 0.03145 6.88725) (end 0.0106 6.956) (layer "Dwgs.User") (width 0.1))
-    (fp_arc (start 5.5923 -6.922) (mid 5.6479 -6.876405) (end 5.6023 -6.8209) (layer "Dwgs.User") (width 0.1))
+    (fp_arc (start 5.5923 -6.922) (mid 5.6478 -6.876495) (end 5.6023 -6.8209) (layer "Dwgs.User") (width 0.1))
     (fp_arc (start 6.1966 -7.4152) (mid 6.140996 -7.36951) (end 6.0955 -7.4252) (layer "Dwgs.User") (width 0.1))
     (fp_arc (start 8.89 -8.8887) (mid 10.236107 -8.331107) (end 10.7937 -6.985) (layer "Dwgs.User") (width 0.1))
@@
   (arc (start 151.5 107.5) (mid 151.207107 106.792893) (end 150.5 106.5) (width 0.25) (layer "B.Cu") (net 42))
   (arc (start 149.5 106.5) (mid 148.792893 106.207107) (end 148.5 105.5) (width 0.25) (layer "B.Cu") (net 42))
-  (segment (start 146.5 125) (end 154 125) (width 0.25) (layer "B.Cu") (net 43))
-  (segment (start 146.5 124) (end 146.5 125) (width 0.25) (layer "B.Cu") (net 43))
-  (segment (start 154 125) (end 154 119) (width 0.25) (layer "B.Cu") (net 43))
-  (segment (start 146.43063 123.93063) (end 146.5 124) (width 0.25) (layer "B.Cu") (net 43))
-  (segment (start 172.05 119) (end 172.05 124.85563) (width 0.25) (layer "B.Cu") (net 43))
-  (segment (start 154 119) (end 172.05 119) (width 0.25) (layer "B.Cu") (net 43))
-  (segment (start 144 123.93063) (end 146.43063 123.93063) (width 0.25) (layer "B.Cu") (net 43))
+  (segment (start 144 125) (end 144 123.93063) (width 0.25) (layer "B.Cu") (net 43))
+  (segment (start 154 120) (end 154 125) (width 0.25) (layer "B.Cu") (net 43))
+  (segment (start 153 126) (end 145 126) (width 0.25) (layer "B.Cu") (net 43))
+  (segment (start 172.05 124.85563) (end 172.05 120) (width 0.25) (layer "B.Cu") (net 43))
+  (segment (start 171.05 119) (end 155 119) (width 0.25) (layer "B.Cu") (net 43))
+  (arc (start 155 119) (mid 154.292893 119.292893) (end 154 120) (width 0.25) (layer "B.Cu") (net 43))
+  (arc (start 153 126) (mid 153.707107 125.707107) (end 154 125) (width 0.25) (layer "B.Cu") (net 43))
+  (arc (start 145 126) (mid 144.292893 125.707107) (end 144 125) (width 0.25) (layer "B.Cu") (net 43))
+  (arc (start 172.05 120) (mid 171.757107 119.292893) (end 171.05 119) (width 0.25) (layer "B.Cu") (net 43))
   (segment (start 159.998446 117.001552) (end 159.988235 123.58063) (width 0.25) (layer "F.Cu") (net 44))
   (segment (start 150 81.67) (end 148.73 80.4) (width 0.25) (layer "F.Cu") (net 44))
@@
   (arc (start 149.5 103.5) (mid 148.792893 103.792893) (end 148.5 104.5) (width 0.25) (layer "F.Cu") (net 45))
   (arc (start 156 118) (mid 155.707107 117.292893) (end 155 117) (width 0.25) (layer "F.Cu") (net 45))
-  (segment (start 142 122) (end 142.06937 121.93063) (width 0.25) (layer "B.Cu") (net 45))
+  (segment (start 144 121.93063) (end 143.10063 121.93063) (width 0.25) (layer "B.Cu") (net 45))
   (segment (start 157.488235 127.28063) (end 155.988235 127.28063) (width 0.25) (layer "B.Cu") (net 45))
-  (segment (start 142.28063 127.28063) (end 142 127) (width 0.25) (layer "B.Cu") (net 45))
   (segment (start 157.488235 127.28063) (end 163.688235 127.28063) (width 0.25) (layer "B.Cu") (net 45))
-  (segment (start 142.06937 121.93063) (end 144 121.93063) (width 0.25) (layer "B.Cu") (net 45))
-  (segment (start 155.988235 127.28063) (end 142.28063 127.28063) (width 0.25) (layer "B.Cu") (net 45))
-  (segment (start 142 127) (end 142 122) (width 0.25) (layer "B.Cu") (net 45))
+  (segment (start 155.988235 127.28063) (end 143.10063 127.28063) (width 0.25) (layer "B.Cu") (net 45))
+  (segment (start 142.10063 122.93063) (end 142.10063 126.28063) (width 0.25) (layer "B.Cu") (net 45))
+  (arc (start 142.10063 126.28063) (mid 142.393523 126.987737) (end 143.10063 127.28063) (width 0.25) (layer "B.Cu") (net 45))
+  (arc (start 142.10063 122.93063) (mid 142.393523 122.223523) (end 143.10063 121.93063) (width 0.25) (layer "B.Cu") (net 45))
   (zone (net 0) (net_name "") (layer "F.Cu") (hatch edge 0.508)
     (connect_pads (clearance 0.508))
